Commit message: add camera

File: urdf/camera.urdf.xacro (robot description, xacro)
@@ -5,5 +5,5 @@
 <!-- reference: https://qiita.com/srs/items/7d78f9ad21a0e61f5bff -->
 <!-- gazebo official: http://gazebosim.org/tutorials?tut=ros_gzplugins -->
-    <!-- <link name="camera">
+    <link name="camera_link">
         <visual>
             <geometry>
@@ -18,10 +18,45 @@
         </inertial>
     </link>
-    <joint name="${name}_sensor_joint" type="fixed">
-        <parent link=""/>
-        <child link=""/>
-        <origin xyz="" rpy=""/>
+    <joint name="$camera_joint" type="fixed">
+        <parent link="base_link"/>
+        <child link="camera_link"/>
+        <origin xyz="0 0.060 0.055" rpy="0 0 0"/>
     </joint>
-    <gazebo reference="${name}_sensor">
-    </gazebo> -->
+    <gazebo reference="camera_link">
+      <sensor type="camera" name="camera_link">
+        <update_rate>10.0</update_rate>
+        <camera name="camera_link">
+          <pose>0 0 0 0 0 ${radians(90)}</pose>
+          <horizontal_fov>1.3962634</horizontal_fov>
+          <image>
+            <width>800</width>
+            <height>600</height>
+            <format>R8G8B8</format>
+          </image>
+          <clip>
+            <near>0.02</near>
+            <far>300</far>
+          </clip>
+          <noise>
+            <type>gaussian</type>
+            <mean>0.0</mean>
+            <stddev>0.007</stddev>
+          </noise>
+        </camera>
+        <plugin name="camera_controller" filename="libgazebo_ros_camera.so">
+          <alwaysOn>true</alwaysOn>
+          <updateRate>0.0</updateRate>
+          <cameraName>camera</cameraName>
+          <imageTopicName>image_raw</imageTopicName>
+          <cameraInfoTopicName>camera_info</cameraInfoTopicName>
+          <frameName>camera_link</frameName>
+          <hackBaseline>0.0</hackBaseline>
+          <distortionK1>0.0</distortionK1>
+          <distortionK2>0.0</distortionK2>
+          <distortionK3>0.0</distortionK3>
+          <distortionT1>0.0</distortionT1>
+          <distortionT2>0.0</distortionT2>
+        </plugin>
+      </sensor>
+    </gazebo>
 </robot>
